Commit message: update urdf

File: Assets/urdf/arm.urdf (robot description, URDF)
Before this commit: robot arm, 5 links, 4 joints
Joints:
- removed joint base_stick1_joint
- removed joint stick1_stick2_joint
- removed joint stick2_stick3_joint
- removed joint stick3_stick4_joint
- added joint 팔_관절1: type revolute, parent stick1, child stick2, origin xyz=0.0 0.0 1 rpy=0.0 0.0 0.0, axis 1 0 0, limit lower=-1.57 upper=1.57 effort=1000 velocity=5.0
- added joint 팔_관절2: type revolute, parent stick2, child stick3, origin xyz=0.0 0.0 1 rpy=0.0 0.0 0.0, axis 1 0 0, limit lower=-1.57 upper=1.57 effort=1000 velocity=5.0
- added joint 팔_길이조절: type prismatic, parent stick3, child stick4, origin xyz=0.0 0.0 0.5 rpy=0.0 0.0 0.0, axis 0 0 1, limit lower=-0.5 upper=0.5 effort=1000 velocity=5.0
- added joint 팔_회전: type revolute, parent main_base, child stick1, origin xyz=0.0 0.0 0.0 rpy=0.0 0.0 0.0, axis 0 0 1, limit lower=-3.14 upper=3.14 effort=1000 velocity=0

File: Assets/urdf/combine.urdf (robot description, URDF)
Before this commit: robot combine, 0 links, 1 joints
Links:
- added link base_link; visual mesh filename=../meshes/base.stl scale=0.01 0.01 0.01
- added link finger_1_link0; visual mesh filename=../meshes/finger0.stl scale=0.01 0.01 0.01
- added link finger_1_link1; visual mesh filename=../meshes/finger1.stl scale=0.01 0.01 0.01
- added link finger_1_link2; visual mesh filename=../meshes/link.stl scale=0.01 0.01 0.01
- added link finger_1_link3; visual mesh filename=../meshes/finger2.stl scale=0.01 0.01 0.01
- added link finger_1_link4; visual mesh filename=../meshes/finger3.stl scale=0.01 0.01 0.01
- added link finger_2_link0; visual mesh filename=../meshes/finger0.stl scale=0.01 0.01 0.01
- added link finger_2_link1; visual mesh filename=../meshes/finger1.stl scale=0.01 0.01 0.01
- added link finger_2_link2; visual mesh filename=../meshes/link.stl scale=0.01 0.01 0.01
- added link finger_2_link3; visual mesh filename=../meshes/finger2.stl scale=0.01 0.01 0.01
- added link finger_2_link4; visual mesh filename=../meshes/finger3.stl scale=0.01 0.01 0.01
- added link finger_3_link0; visual mesh filename=../meshes/finger0.stl scale=0.01 0.01 0.01
- added link finger_3_link1; visual mesh filename=../meshes/finger1.stl scale=0.01 0.01 0.01
- added link finger_3_link2; visual mesh filename=../meshes/link.stl scale=0.01 0.01 0.01
- added link finger_3_link3; visual mesh filename=../meshes/finger2.stl scale=0.01 0.01 0.01
- added link finger_3_link4; visual mesh filename=../meshes/finger3.stl scale=0.01 0.01 0.01
- added link main_base; visual cylinder length=0.2 radius=0.6
- added link palm_link; visual mesh filename=../meshes/housing.stl scale=0.01 0.01 0.01
- added link stick1; visual cylinder length=1 radius=0.2
- added link stick2; visual cylinder length=1 radius=0.2
- added link stick3; visual cylinder length=1 radius=0.2
- added link stick4; visual cylinder length=1 radius=0.15
Joints:
- removed joint joint_name
- added joint 검지_롤: type revolute, parent finger_2_link1, child finger_2_link2, origin xyz=0.123 0.005 0.293 rpy=0 1.57 0, axis 0 0 1, limit lower=-1.57 upper=1.57 effort=1000 velocity=5.027
- added joint 검지_연결부: type fixed, parent base_link, child finger_2_link0, origin xyz=-0.05 -0.196 0.142 rpy=0 0 3.14, axis 0 0 1
- added joint 검지_요: type revolute, parent finger_2_link0, child finger_2_link1, origin xyz=0.07 0 0.284 rpy=0 0 0, axis 0 0 1, limit lower=0 upper=0.785 effort=1000 velocity=5.027
- added joint 검지_피치1: type revolute, parent finger_2_link2, child finger_2_link3, origin xyz=-0.1 0 0.2 rpy=1.57 0 0, axis 0 0 1, limit lower=0 upper=1.57 effort=1000 velocity=5.027
- added joint 검지_피치2: type revolute, parent finger_2_link3, child finger_2_link4, origin xyz=0 0.445 0 rpy=0 0 0, axis 0 0 1, limit lower=0 upper=1.57 effort=1000 velocity=5.027
- added joint 손목_회전: type revolute, parent stick4, child base_link, origin xyz=0.0 0.0 1.2 rpy=0.0 0.0 0.0, axis 0.0 0.0 1.0, limit lower=-3.14 upper=3.14 effort=1000 velocity=5.0
- added joint 손바닥_연결부: type fixed, parent base_link, child palm_link, origin xyz=0 0 0.7 rpy=0 0 0, axis 0 0 1
- added joint 엄지_롤: type revolute, parent finger_1_link1, child finger_1_link2, origin xyz=0.123 0.005 0.293 rpy=0 1.57 0, axis 0 0 1, limit lower=-1.57 upper=1.57 effort=1000 velocity=5.027
- added joint 엄지_연결부: type fixed, parent base_link, child finger_1_link0, origin xyz=0.098 0 0.142 rpy=0 0 0, axis 0 0 1
- added joint 엄지_요: type revolute, parent finger_1_link0, child finger_1_link1, origin xyz=0.07 0 0.284 rpy=0 0 0, axis 0 0 1, limit lower=-0.785 upper=0.785 effort=1000 velocity=5.027
- added joint 엄지_피치1: type revolute, parent finger_1_link2, child finger_1_link3, origin xyz=-0.1 0 0.2 rpy=1.57 0 0, axis 0 0 1, limit lower=0 upper=1.57 effort=1000 velocity=5.027
- added joint 엄지_피치2: type revolute, parent finger_1_link3, child finger_1_link4, origin xyz=0 0.445 0 rpy=0 0 0, axis 0 0 1, limit lower=0 upper=1.57 effort=1000 velocity=5.027
- added joint 중지_롤: type revolute, parent finger_3_link1, child finger_3_link2, origin xyz=0.123 +0.005 0.293 rpy=0 1.57 0, axis 0 0 1, limit lower=-1.57 upper=1.57 effort=1000 velocity=5.027
- added joint 중지_연결부: type fixed, parent base_link, child finger_3_link0, origin xyz=-0.05 0.196 0.142 rpy=0 0 3.14, axis 0 0 1
- added joint 중지_요: type revolute, parent finger_3_link0, child finger_3_link1, origin xyz=0.07 0 0.284 rpy=0 0 0, axis 0 0 1, limit lower=-0.785 upper=0 effort=1000 velocity=5.027
- added joint 중지_피치1: type revolute, parent finger_3_link2, child finger_3_link3, origin xyz=-0.1 0 0.2 rpy=1.57 0 0, axis 0 0 1, limit lower=0 upper=1.57 effort=1000 velocity=5.027
- added joint 중지_피치2: type revolute, parent finger_3_link3, child finger_3_link4, origin xyz=0 0.445 0 rpy=0 0 0, axis 0 0 1, limit lower=0 upper=1.57 effort=1000 velocity=5.027
- added joint 팔_관절1: type revolute, parent stick1, child stick2, origin xyz=0.0 0.0 1 rpy=0.0 0.0 0.0, axis 1 0 0, limit lower=-1.57 upper=1.57 effort=1000 velocity=5.0
- added joint 팔_관절2: type revolute, parent stick2, child stick3, origin xyz=0.0 0.0 1 rpy=0.0 0.0 0.0, axis 1 0 0, limit lower=-1.57 upper=1.57 effort=1000 velocity=5.0
- added joint 팔_길이조절: type prismatic, parent stick3, child stick4, origin xyz=0.0 0.0 0.5 rpy=0.0 0.0 0.0, axis 0 0 1, limit lower=-0.5 upper=0.5 effort=1000 velocity=5.0
- added joint 팔_회전: type revolute, parent main_base, child stick1, origin xyz=0.0 0.0 0.0 rpy=0.0 0.0 0.0, axis 0 0 1, limit lower=-3.14 upper=3.14 effort=1000 velocity=0

File: Assets/urdf/hand.urdf (robot description, URDF)
Before this commit: robot robot_hand, 17 links, 16 joints
Joints:
- removed joint finger_1_joint0
- removed joint finger_1_joint1
- removed joint finger_1_joint2
- removed joint finger_1_joint3
- removed joint finger_1_joint4
- removed joint finger_2_joint0
- removed joint finger_2_joint1
- removed joint finger_2_joint2
- removed joint finger_2_joint3
- removed joint finger_2_joint4
- removed joint finger_3_joint0
- removed joint finger_3_joint1
- removed joint finger_3_joint2
- removed joint finger_3_joint3
- removed joint finger_3_joint4
- removed joint palm_joint
- added joint 검지_롤: type revolute, parent finger_2_link1, child finger_2_link2, origin xyz=0.123 0.005 0.293 rpy=0 1.57 0, axis 0 0 1, limit lower=-1.57 upper=1.57 effort=1000 velocity=5.027
- added joint 검지_연결부: type fixed, parent base_link, child finger_2_link0, origin xyz=-0.05 -0.196 0.142 rpy=0 0 3.14, axis 0 0 1
- added joint 검지_요: type revolute, parent finger_2_link0, child finger_2_link1, origin xyz=0.07 0 0.284 rpy=0 0 0, axis 0 0 1, limit lower=0 upper=0.785 effort=1000 velocity=5.027
- added joint 검지_피치1: type revolute, parent finger_2_link2, child finger_2_link3, origin xyz=-0.1 0 0.2 rpy=1.57 0 0, axis 0 0 1, limit lower=0 upper=1.57 effort=1000 velocity=5.027
- added joint 검지_피치2: type revolute, parent finger_2_link3, child finger_2_link4, origin xyz=0 0.445 0 rpy=0 0 0, axis 0 0 1, limit lower=0 upper=1.57 effort=1000 velocity=5.027
- added joint 손바닥_연결부: type fixed, parent base_link, child palm_link, origin xyz=0 0 0.7 rpy=0 0 0, axis 0 0 1
- added joint 엄지_롤: type revolute, parent finger_1_link1, child finger_1_link2, origin xyz=0.123 0.005 0.293 rpy=0 1.57 0, axis 0 0 1, limit lower=-1.57 upper=1.57 effort=1000 velocity=5.027
- added joint 엄지_연결부: type fixed, parent base_link, child finger_1_link0, origin xyz=0.098 0 0.142 rpy=0 0 0, axis 0 0 1
- added joint 엄지_요: type revolute, parent finger_1_link0, child finger_1_link1, origin xyz=0.07 0 0.284 rpy=0 0 0, axis 0 0 1, limit lower=-0.785 upper=0.785 effort=1000 velocity=5.027
- added joint 엄지_피치1: type revolute, parent finger_1_link2, child finger_1_link3, origin xyz=-0.1 0 0.2 rpy=1.57 0 0, axis 0 0 1, limit lower=0 upper=1.57 effort=1000 velocity=5.027
- added joint 엄지_피치2: type revolute, parent finger_1_link3, child finger_1_link4, origin xyz=0 0.445 0 rpy=0 0 0, axis 0 0 1, limit lower=0 upper=1.57 effort=1000 velocity=5.027
- added joint 중지_롤: type revolute, parent finger_3_link1, child finger_3_link2, origin xyz=0.123 +0.005 0.293 rpy=0 1.57 0, axis 0 0 1, limit lower=-1.57 upper=1.57 effort=1000 velocity=5.027
- added joint 중지_연결부: type fixed, parent base_link, child finger_3_link0, origin xyz=-0.05 0.196 0.142 rpy=0 0 3.14, axis 0 0 1
- added joint 중지_요: type revolute, parent finger_3_link0, child finger_3_link1, origin xyz=0.07 0 0.284 rpy=0 0 0, axis 0 0 1, limit lower=-0.785 upper=0 effort=1000 velocity=5.027
- added joint 중지_피치1: type revolute, parent finger_3_link2, child finger_3_link3, origin xyz=-0.1 0 0.2 rpy=1.57 0 0, axis 0 0 1, limit lower=0 upper=1.57 effort=1000 velocity=5.027
- added joint 중지_피치2: type revolute, parent finger_3_link3, child finger_3_link4, origin xyz=0 0.445 0 rpy=0 0 0, axis 0 0 1, limit lower=0 upper=1.57 effort=1000 velocity=5.027

Commit message: update urdf

File: Assets/urdf/arm.urdf (robot description, URDF)
Before this commit: robot arm, 5 links, 4 joints
Joints:
- removed joint 팔_관절1
- removed joint 팔_관절2
- removed joint 팔_길이조절
- removed joint 팔_회전
- added joint M1_A0: type revolute, parent main_base, child stick1, origin xyz=0.0 0.0 0.0 rpy=0.0 0.0 0.0, axis 0 0 1, limit lower=-3.14 upper=3.14 effort=1000 velocity=0
- added joint S1_A0: type revolute, parent stick1, child stick2, origin xyz=0.0 0.0 1 rpy=0.0 0.0 0.0, axis 1 0 0, limit lower=-1.57 upper=1.57 effort=1000 velocity=5.0
- added joint S2_A0: type revolute, parent stick2, child stick3, origin xyz=0.0 0.0 1 rpy=0.0 0.0 0.0, axis 1 0 0, limit lower=-1.57 upper=1.57 effort=1000 velocity=5.0
- added joint S3_A0: type prismatic, parent stick3, child stick4, origin xyz=0.0 0.0 0.5 rpy=0.0 0.0 0.0, axis 0 0 1, limit lower=-0.5 upper=0.5 effort=1000 velocity=5.0

File: Assets/urdf/combine.urdf (robot description, URDF)
Before this commit: robot combine, 22 links, 21 joints
Joints:
- removed joint 검지_롤
- removed joint 검지_연결부
- removed joint 검지_요
- removed joint 검지_피치1
- removed joint 검지_피치2
- removed joint 손목_회전
- removed joint 손바닥_연결부
- removed joint 엄지_롤
- removed joint 엄지_연결부
- removed joint 엄지_요
- removed joint 엄지_피치1
- removed joint 엄지_피치2
- removed joint 중지_롤
- removed joint 중지_연결부
- removed joint 중지_요
- removed joint 중지_피치1
- removed joint 중지_피치2
- removed joint 팔_관절1
- removed joint 팔_관절2
- removed joint 팔_길이조절
- removed joint 팔_회전
- added joint FIXED96: type fixed, parent base_link, child finger_3_link0, origin xyz=-0.05 0.196 0.142 rpy=0 0 3.14, axis 0 0 1
- added joint FIXED97: type fixed, parent base_link, child finger_2_link0, origin xyz=-0.05 -0.196 0.142 rpy=0 0 3.14, axis 0 0 1
- added joint FIXED98: type fixed, parent base_link, child finger_1_link0, origin xyz=0.098 0 0.142 rpy=0 0 0, axis 0 0 1
- added joint FIXED99: type fixed, parent base_link, child palm_link, origin xyz=0 0 0.7 rpy=0 0 0, axis 0 0 1
- added joint M1_A0: type revolute, parent main_base, child stick1, origin xyz=0.0 0.0 0.0 rpy=0.0 0.0 0.0, axis 0 0 1, limit lower=-3.14 upper=3.14 effort=1000 velocity=0
- added joint P1_F1: type revolute, parent finger_1_link2, child finger_1_link3, origin xyz=-0.1 0 0.2 rpy=1.57 0 0, axis 0 0 1, limit lower=0 upper=1.57 effort=1000 velocity=5.027
- added joint P1_F2: type revolute, parent finger_2_link2, child finger_2_link3, origin xyz=-0.1 0 0.2 rpy=1.57 0 0, axis 0 0 1, limit lower=0 upper=1.57 effort=1000 velocity=5.027
- added joint P1_F3: type revolute, parent finger_3_link2, child finger_3_link3, origin xyz=-0.1 0 0.2 rpy=1.57 0 0, axis 0 0 1, limit lower=0 upper=1.57 effort=1000 velocity=5.027
- added joint P2_F1: type revolute, parent finger_1_link3, child finger_1_link4, origin xyz=0 0.445 0 rpy=0 0 0, axis 0 0 1, limit lower=0 upper=1.57 effort=1000 velocity=5.027
- added joint P2_F2: type revolute, parent finger_2_link3, child finger_2_link4, origin xyz=0 0.445 0 rpy=0 0 0, axis 0 0 1, limit lower=0 upper=1.57 effort=1000 velocity=5.027
- added joint P2_F3: type revolute, parent finger_3_link3, child finger_3_link4, origin xyz=0 0.445 0 rpy=0 0 0, axis 0 0 1, limit lower=0 upper=1.57 effort=1000 velocity=5.027
- added joint R1_F1: type revolute, parent finger_1_link1, child finger_1_link2, origin xyz=0.123 0.005 0.293 rpy=0 1.57 0, axis 0 0 1, limit lower=-1.57 upper=1.57 effort=1000 velocity=5.027
- added joint R1_F2: type revolute, parent finger_2_link1, child finger_2_link2, origin xyz=0.123 0.005 0.293 rpy=0 1.57 0, axis 0 0 1, limit lower=-1.57 upper=1.57 effort=1000 velocity=5.027
- added joint R1_F3: type revolute, parent finger_3_link1, child finger_3_link2, origin xyz=0.123 +0.005 0.293 rpy=0 1.57 0, axis 0 0 1, limit lower=-1.57 upper=1.57 effort=1000 velocity=5.027
- added joint S1_A0: type revolute, parent stick1, child stick2, origin xyz=0.0 0.0 1 rpy=0.0 0.0 0.0, axis 1 0 0, limit lower=-1.57 upper=1.57 effort=1000 velocity=5.0
- added joint S2_A0: type revolute, parent stick2, child stick3, origin xyz=0.0 0.0 1 rpy=0.0 0.0 0.0, axis 1 0 0, limit lower=-1.57 upper=1.57 effort=1000 velocity=5.0
- added joint S3_A0: type prismatic, parent stick3, child stick4, origin xyz=0.0 0.0 0.5 rpy=0.0 0.0 0.0, axis 0 0 1, limit lower=-0.5 upper=0.5 effort=1000 velocity=5.0
- added joint S4_A0: type revolute, parent stick4, child base_link, origin xyz=0.0 0.0 1.2 rpy=0.0 0.0 0.0, axis 0.0 0.0 1.0, limit lower=-3.14 upper=3.14 effort=1000 velocity=5.0
- added joint Y1_F1: type revolute, parent finger_1_link0, child finger_1_link1, origin xyz=0.07 0 0.284 rpy=0 0 0, axis 0 0 1, limit lower=-0.785 upper=0.785 effort=1000 velocity=5.027
- added joint Y1_F2: type revolute, parent finger_2_link0, child finger_2_link1, origin xyz=0.07 0 0.284 rpy=0 0 0, axis 0 0 1, limit lower=0 upper=0.785 effort=1000 velocity=5.027
- added joint Y1_F3: type revolute, parent finger_3_link0, child finger_3_link1, origin xyz=0.07 0 0.284 rpy=0 0 0, axis 0 0 1, limit lower=-0.785 upper=0 effort=1000 velocity=5.027

File: Assets/urdf/hand.urdf (robot description, URDF)
Before this commit: robot robot_hand, 17 links, 16 joints
Joints:
- removed joint 검지_롤
- removed joint 검지_연결부
- removed joint 검지_요
- removed joint 검지_피치1
- removed joint 검지_피치2
- removed joint 손바닥_연결부
- removed joint 엄지_롤
- removed joint 엄지_연결부
- removed joint 엄지_요
- removed joint 엄지_피치1
- removed joint 엄지_피치2
- removed joint 중지_롤
- removed joint 중지_연결부
- removed joint 중지_요
- removed joint 중지_피치1
- removed joint 중지_피치2
- added joint FIXED96: type fixed, parent base_link, child finger_3_link0, origin xyz=-0.05 0.196 0.142 rpy=0 0 3.14, axis 0 0 1
- added joint FIXED97: type fixed, parent base_link, child finger_2_link0, origin xyz=-0.05 -0.196 0.142 rpy=0 0 3.14, axis 0 0 1
- added joint FIXED98: type fixed, parent base_link, child finger_1_link0, origin xyz=0.098 0 0.142 rpy=0 0 0, axis 0 0 1
- added joint FIXED99: type fixed, parent base_link, child palm_link, origin xyz=0 0 0.7 rpy=0 0 0, axis 0 0 1
- added joint P1_F1: type revolute, parent finger_1_link2, child finger_1_link3, origin xyz=-0.1 0 0.2 rpy=1.57 0 0, axis 0 0 1, limit lower=0 upper=1.57 effort=1000 velocity=5.027
- added joint P1_F2: type revolute, parent finger_2_link2, child finger_2_link3, origin xyz=-0.1 0 0.2 rpy=1.57 0 0, axis 0 0 1, limit lower=0 upper=1.57 effort=1000 velocity=5.027
- added joint P1_F3: type revolute, parent finger_3_link2, child finger_3_link3, origin xyz=-0.1 0 0.2 rpy=1.57 0 0, axis 0 0 1, limit lower=0 upper=1.57 effort=1000 velocity=5.027
- added joint P2_F1: type revolute, parent finger_1_link3, child finger_1_link4, origin xyz=0 0.445 0 rpy=0 0 0, axis 0 0 1, limit lower=0 upper=1.57 effort=1000 velocity=5.027
- added joint P2_F2: type revolute, parent finger_2_link3, child finger_2_link4, origin xyz=0 0.445 0 rpy=0 0 0, axis 0 0 1, limit lower=0 upper=1.57 effort=1000 velocity=5.027
- added joint P2_F3: type revolute, parent finger_3_link3, child finger_3_link4, origin xyz=0 0.445 0 rpy=0 0 0, axis 0 0 1, limit lower=0 upper=1.57 effort=1000 velocity=5.027
- added joint R1_F1: type revolute, parent finger_1_link1, child finger_1_link2, origin xyz=0.123 0.005 0.293 rpy=0 1.57 0, axis 0 0 1, limit lower=-1.57 upper=1.57 effort=1000 velocity=5.027
- added joint R1_F2: type revolute, parent finger_2_link1, child finger_2_link2, origin xyz=0.123 0.005 0.293 rpy=0 1.57 0, axis 0 0 1, limit lower=-1.57 upper=1.57 effort=1000 velocity=5.027
- added joint R1_F3: type revolute, parent finger_3_link1, child finger_3_link2, origin xyz=0.123 +0.005 0.293 rpy=0 1.57 0, axis 0 0 1, limit lower=-1.57 upper=1.57 effort=1000 velocity=5.027
- added joint Y1_F1: type revolute, parent finger_1_link0, child finger_1_link1, origin xyz=0.07 0 0.284 rpy=0 0 0, axis 0 0 1, limit lower=-0.785 upper=0.785 effort=1000 velocity=5.027
- added joint Y1_F2: type revolute, parent finger_2_link0, child finger_2_link1, origin xyz=0.07 0 0.284 rpy=0 0 0, axis 0 0 1, limit lower=0 upper=0.785 effort=1000 velocity=5.027
- added joint Y1_F3: type revolute, parent finger_3_link0, child finger_3_link1, origin xyz=0.07 0 0.284 rpy=0 0 0, axis 0 0 1, limit lower=-0.785 upper=0 effort=1000 velocity=5.027
